File: PCB/manual_input.kicad_sch (KiCad schematic)
At the start: 3 parts

Commit message: :wrench: Assign footprints to all symbols
Parts:
- C?: footprint (none) -> Capacitor_THT:C_Disc_D4.3mm_W1.9mm_P5.00mm
- R?: footprint (none) -> Resistor_THT:R_Axial_DIN0207_L6.3mm_D2.5mm_P7.62mm_Horizontal
Changed lines of the file:
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@@
       (effects (font (size 1.27 1.27)) (justify left))
     )
-    (property "Footprint" "" (at 58.7248 40.64 0)
+    (property "Footprint" "Capacitor_THT:C_Disc_D4.3mm_W1.9mm_P5.00mm" (at 58.7248 40.64 0)
       (effects (font (size 1.27 1.27)) hide)
     )
@@
       (effects (font (size 1.27 1.27)))
     )
-    (property "Footprint" "" (at 53.34 41.148 90)
+    (property "Footprint" "Resistor_THT:R_Axial_DIN0207_L6.3mm_D2.5mm_P7.62mm_Horizontal" (at 53.34 41.148 90)
       (effects (font (size 1.27 1.27)) hide)
     )

Commit message: :rocket: Update the revision number
Other:
- company: (none) -> moPsy
- title: (none) -> Manual Gate/Trigger Source
Changed lines of the file:
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@@
 (kicad_sch (version 20230121) (generator eeschema)
   (paper "A4")
+  (title_block
+    (title "Manual Gate/Trigger Source")
+    (rev "v2")
+    (company "moPsy")
+  )
   (junction (at 59.69 39.37) (diameter 0) (color 0 0 0 0)
   )
